Commit message: Update robot configuration and improve arm gain profiles

File: assets/my_B2Arx/my_robot.urdf (robot description, URDF)
Before this commit: robot my_robot, 46 links, 45 joints
Joints:
- joint d435i_mount: origin xyz=0.06 0 0.07 rpy=0 0.2618 0 -> xyz=0.06 0 0.10 rpy=0 0.523599 0

Commit message: Add new materials and gamepad mapping script

File: assets/my_B2Arx/my_robot.urdf (robot description, URDF)
Before this commit: robot my_robot, 46 links, 45 joints
Links:
- removed link d435i_link
Joints:
- removed joint d435i_mount
